File: hardware/hall_effect_sensor/hall_effect_sensor.kicad_pcb (KiCad board)
At the start: 2 copper layers, 14 x 10 mm, 4 parts, among them J1 HALL, U1 A1369xUA-10

Commit message: Updating board to include mounting holes.
Routing:
- net (no net): vias 0 -> 4
Other:
- board size 14 x 10 mm -> 15 x 16 mm
- board text added: "2020- 03-08"
- board text added: "kazatsky HESense"
Changed lines of the file:
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@@
   (general
     (thickness 1.6)
-    (drawings 10)
-    (tracks 18)
+    (drawings 12)
+    (tracks 22)
     (zones 0)
     (modules 4)
@@
       (effects (font (size 1 1) (thickness 0.15)))
     )
+    (fp_line (start -0.635 -1.27) (end 1.27 -1.27) (layer F.Fab) (width 0.1))
+    (fp_line (start 1.27 -1.27) (end 1.27 6.35) (layer F.Fab) (width 0.1))
+    (fp_line (start 1.27 6.35) (end -1.27 6.35) (layer F.Fab) (width 0.1))
+    (fp_line (start -1.27 6.35) (end -1.27 -0.635) (layer F.Fab) (width 0.1))
+    (fp_line (start -1.27 -0.635) (end -0.635 -1.27) (layer F.Fab) (width 0.1))
+    (fp_line (start -1.33 6.41) (end 1.33 6.41) (layer F.SilkS) (width 0.12))
+    (fp_line (start -1.33 1.27) (end -1.33 6.41) (layer F.SilkS) (width 0.12))
+    (fp_line (start 1.33 1.27) (end 1.33 6.41) (layer F.SilkS) (width 0.12))
+    (fp_line (start -1.33 1.27) (end 1.33 1.27) (layer F.SilkS) (width 0.12))
+    (fp_line (start -1.33 0) (end -1.33 -1.33) (layer F.SilkS) (width 0.12))
+    (fp_line (start -1.33 -1.33) (end 0 -1.33) (layer F.SilkS) (width 0.12))
+    (fp_line (start -1.8 -1.8) (end -1.8 6.85) (layer F.CrtYd) (width 0.05))
+    (fp_line (start -1.8 6.85) (end 1.8 6.85) (layer F.CrtYd) (width 0.05))
+    (fp_line (start 1.8 6.85) (end 1.8 -1.8) (layer F.CrtYd) (width 0.05))
     (fp_line (start 1.8 -1.8) (end -1.8 -1.8) (layer F.CrtYd) (width 0.05))
-    (fp_line (start 1.8 6.85) (end 1.8 -1.8) (layer F.CrtYd) (width 0.05))
-    (fp_line (start -1.8 6.85) (end 1.8 6.85) (layer F.CrtYd) (width 0.05))
-    (fp_line (start -1.8 -1.8) (end -1.8 6.85) (layer F.CrtYd) (width 0.05))
-    (fp_line (start -1.33 -1.33) (end 0 -1.33) (layer F.SilkS) (width 0.12))
-    (fp_line (start -1.33 0) (end -1.33 -1.33) (layer F.SilkS) (width 0.12))
-    (fp_line (start -1.33 1.27) (end 1.33 1.27) (layer F.SilkS) (width 0.12))
-    (fp_line (start 1.33 1.27) (end 1.33 6.41) (layer F.SilkS) (width 0.12))
-    (fp_line (start -1.33 1.27) (end -1.33 6.41) (layer F.SilkS) (width 0.12))
-    (fp_line (start -1.33 6.41) (end 1.33 6.41) (layer F.SilkS) (width 0.12))
-    (fp_line (start -1.27 -0.635) (end -0.635 -1.27) (layer F.Fab) (width 0.1))
-    (fp_line (start -1.27 6.35) (end -1.27 -0.635) (layer F.Fab) (width 0.1))
-    (fp_line (start 1.27 6.35) (end -1.27 6.35) (layer F.Fab) (width 0.1))
-    (fp_line (start 1.27 -1.27) (end 1.27 6.35) (layer F.Fab) (width 0.1))
-    (fp_line (start -0.635 -1.27) (end 1.27 -1.27) (layer F.Fab) (width 0.1))
     (fp_text user %R (at 0 2.54 90) (layer F.Fab)
       (effects (font (size 1 1) (thickness 0.15)))
@@
       (effects (font (size 1 1) (thickness 0.15)))
     )
+    (fp_line (start 3.57 1.05) (end 3.57 -1.05) (layer F.CrtYd) (width 0.05))
+    (fp_line (start -1.03 1.05) (end 3.57 1.05) (layer F.CrtYd) (width 0.05))
+    (fp_line (start -1.03 -1.05) (end -1.03 1.05) (layer F.CrtYd) (width 0.05))
+    (fp_line (start 3.57 -1.05) (end -1.03 -1.05) (layer F.CrtYd) (width 0.05))
+    (fp_line (start -0.775 0) (end 0.015 0.79) (layer F.Fab) (width 0.1))
+    (fp_line (start 2.525 0.79) (end 0.015 0.79) (layer F.Fab) (width 0.1))
+    (fp_line (start 3.315 0) (end 2.525 0.79) (layer F.Fab) (width 0.1))
+    (fp_line (start 3.315 -0.73) (end 3.315 0) (layer F.Fab) (width 0.1))
+    (fp_line (start -0.775 -0.73) (end 3.315 -0.73) (layer F.Fab) (width 0.1))
+    (fp_line (start -0.775 0) (end -0.775 -0.73) (layer F.Fab) (width 0.1))
+    (fp_line (start 2.01 -0.85) (end 1.8 -0.85) (layer F.SilkS) (width 0.12))
+    (fp_line (start 2.01 0.91) (end 1.8 0.91) (layer F.SilkS) (width 0.12))
+    (fp_line (start 3.435 -0.85) (end 3.435 0) (layer F.SilkS) (width 0.12))
+    (fp_line (start -0.895 0) (end -0.895 -0.85) (layer F.SilkS) (width 0.12))
     (fp_line (start 3.435 -0.85) (end 3.07 -0.85) (layer F.SilkS) (width 0.12))
-    (fp_line (start -0.895 0) (end -0.895 -0.85) (layer F.SilkS) (width 0.12))
-    (fp_line (start 3.435 -0.85) (end 3.435 0) (layer F.SilkS) (width 0.12))
-    (fp_line (start 2.01 0.91) (end 1.8 0.91) (layer F.SilkS) (width 0.12))
-    (fp_line (start 2.01 -0.85) (end 1.8 -0.85) (layer F.SilkS) (width 0.12))
-    (fp_line (start -0.775 0) (end -0.775 -0.73) (layer F.Fab) (width 0.1))
-    (fp_line (start -0.775 -0.73) (end 3.315 -0.73) (layer F.Fab) (width 0.1))
-    (fp_line (start 3.315 -0.73) (end 3.315 0) (layer F.Fab) (width 0.1))
-    (fp_line (start 3.315 0) (end 2.525 0.79) (layer F.Fab) (width 0.1))
-    (fp_line (start 2.525 0.79) (end 0.015 0.79) (layer F.Fab) (width 0.1))
-    (fp_line (start -0.775 0) (end 0.015 0.79) (layer F.Fab) (width 0.1))
-    (fp_line (start 3.57 -1.05) (end -1.03 -1.05) (layer F.CrtYd) (width 0.05))
-    (fp_line (start -1.03 -1.05) (end -1.03 1.05) (layer F.CrtYd) (width 0.05))
-    (fp_line (start -1.03 1.05) (end 3.57 1.05) (layer F.CrtYd) (width 0.05))
-    (fp_line (start 3.57 1.05) (end 3.57 -1.05) (layer F.CrtYd) (width 0.05))
     (fp_text user %R (at 1.27 0 90) (layer F.Fab)
       (effects (font (size 0.8 0.8) (thickness 0.1)))
@@
       (effects (font (size 1 1) (thickness 0.15)) (justify mirror))
     )
+    (fp_line (start -0.6 0.875) (end 0.6 0.875) (layer B.SilkS) (width 0.15))
     (fp_line (start 0.6 -0.875) (end -0.6 -0.875) (layer B.SilkS) (width 0.15))
-    (fp_line (start -0.6 0.875) (end 0.6 0.875) (layer B.SilkS) (width 0.15))
     (pad 1 smd rect (at -1 0 90) (size 1.79 1.3) (layers B.Cu B.Paste B.Mask)
       (net 1 "Net-(C1-Pad1)"))
@@
       (effects (font (size 1 1) (thickness 0.15)) (justify mirror))
     )
+    (fp_line (start -0.6 0.875) (end 0.6 0.875) (layer B.SilkS) (width 0.15))
     (fp_line (start 0.6 -0.875) (end -0.6 -0.875) (layer B.SilkS) (width 0.15))
-    (fp_line (start -0.6 0.875) (end 0.6 0.875) (layer B.SilkS) (width 0.15))
     (pad 1 smd rect (at -1 0 270) (size 1.79 1.3) (layers B.Cu B.Paste B.Mask)
       (net 1 "Net-(C1-Pad1)"))
@@
     )
   )
-  (gr_line (start 40 49) (end 40 39) (layer Edge.Cuts) (width 0.05))
-  (gr_line (start 54 49) (end 40 49) (layer Edge.Cuts) (width 0.05))
-  (gr_line (start 54 39) (end 54 49) (layer Edge.Cuts) (width 0.05))
-  (gr_line (start 40 39) (end 54 39) (layer Edge.Cuts) (width 0.05))
+  (gr_text "2020-\n03-08" (at 47 50) (layer F.Cu)
+    (effects (font (size 1 1) (thickness 0.25)))
+  )
+  (gr_text "kazatsky\nHESense" (at 43 38) (layer F.Cu)
+    (effects (font (size 1 1) (thickness 0.25)) (justify left))
+  )
+  (gr_line (start 39 52) (end 39 36) (layer Edge.Cuts) (width 0.05))
+  (gr_line (start 54 52) (end 39 52) (layer Edge.Cuts) (width 0.05))
+  (gr_line (start 54 36) (end 54 52) (layer Edge.Cuts) (width 0.05))
+  (gr_line (start 39 36) (end 54 36) (layer Edge.Cuts) (width 0.05))
   (gr_text S (at 41.1 46.8 180) (layer F.Cu)
     (effects (font (size 1.5 1.5) (thickness 0.3)))
@@
     (effects (font (size 1.5 1.5) (thickness 0.3)))
   )
+  (via (at 52 38) (size 3) (drill 2.5) (layers F.Cu B.Cu) (net 0))
+  (via (at 41 38) (size 3) (drill 2.5) (layers F.Cu B.Cu) (net 0))
+  (via (at 41 50) (size 3) (drill 2.5) (layers F.Cu B.Cu) (net 0))
+  (via (at 52 50) (size 3) (drill 2.5) (layers F.Cu B.Cu) (net 0))
   (segment (start 45.634999 44.165001) (end 46.7 43.1) (width 0.45) (layer B.Cu) (net 1))
   (segment (start 43.825001 44.165001) (end 45.634999 44.165001) (width 0.45) (layer B.Cu) (net 1))
